File: PCB/logic.sch (KiCad schematic (older format))
At the start: 45 parts, among them IC1 ATTINY2313-P, IC2 ATTINY2313-P, P1 ISP, P2 CONN_01X05, P3 CONN_01X02, P4 DS18B20 data, Q1 BC817-40, Q2 BC817-40, SW1 UP, SW2 DOWN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

Commit message: Changed the schematic to be on only one board
Parts:
- removed P2: CONN_01X05, Socket_Strips:Socket_Strip_Straight_1x05, symbol CONN_01X05
- added 4V2: ZENER, symbol ZENER
- added BT1: Battery, symbol Battery
- added D5, D6: D, Capacitors_SMD:C_0805_HandSoldering, symbol D
- added P2: 5VDC, symbol CONN_01X02
- added P5: CONN_01X04, symbol CONN_01X04
- added R24: 220R, Resistors_SMD:R_0603_HandSoldering, symbol R
- added R25: 1K, Resistors_SMD:R_0603_HandSoldering, symbol R
- added U1, U2: MOC3023M, DIP-6, symbol MOC3023M
- R16: value 1K -> 220R
Connections:
- net GNDREF: now also 4V2.2 (A), BT1.2, P2.2 (P2), U1.2, U2.2
- net VCC: now also D4.2 (A), R23.1, P2.1 (P1), R25.2; no longer R23.2
- net at R16.2: now also U1.1
- net at IC2.18 ((PCINT6/MISO/DO)PB6): now also R24.1
- net at C4.1, D4.1 (K), IC2.20 (VCC)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: now also D5.1 (K)
- new net: IC2.19 ((PCINT7/USCK/SCK/SCL)PB7), R23.2
- new net: P5.4 (P4), U1.4, U2.4
- new net: P5.2 (P2), U1.6
- new net: R24.2, U2.1
- new net: P5.3 (P3), U2.6
- new net: BT1.1, D5.2 (A), D6.1 (K)
- new net: 4V2.1 (K), D6.2 (A), R25.1
- no-connect marks 11 -> 12
Other:
- note added: "Fan"
- note added: "Heat"
- note added: "N"
- note added: "R"
- moved on the sheet: D4, R23
